File: Pulse_Module.kicad_pcb (KiCad board)
At the start: 2 copper layers, 2 parts, among them CON1 AVR-ISP-10

Commit message: Изменения в CvPCB
Parts:
- added C10: 0.1uF, Capacitors_SMD:C_0402, F.Cu at (144.9, 21.4)
- added C11: 0.1uF, Capacitors_SMD:C_0402, F.Cu at (116.0, 38.4)
- added C12: 0.1uF, Capacitors_SMD:C_0402, F.Cu at (120.2, 32.5)
- added C13: 104, Capacitors_SMD:C_0603_HandSoldering, F.Cu at (77.8, 35.2)
- added C14: 0.1uF, Capacitors_SMD:C_0402, F.Cu at (102.2, 53.0)
- added C15: 0.1uF, Capacitors_SMD:C_0402, F.Cu at (89.8, 66.0)
- added C17: 0.1U, Capacitors_SMD:C_0402, F.Cu at (108.0, 47.1)
- added C18: 0.1uF, Capacitors_SMD:C_0402, F.Cu at (94.5, 59.3)
- added C19: 27pF, Capacitors_SMD:C_0603_HandSoldering, F.Cu at (101.4, 47.3)
- added C2: 0.1uF, Capacitors_SMD:C_0402, F.Cu at (159.0, 10.8)
- added C21: 27pF, Capacitors_SMD:C_0603_HandSoldering, F.Cu at (69.4, 35.2)
- added C22: 27pF, Capacitors_SMD:C_0603_HandSoldering, F.Cu at (73.6, 35.2)
- added C3: 0.1uF, Capacitors_SMD:C_0402, F.Cu at (108.3, 52.6)
- added C4: 27pF, Capacitors_SMD:C_0603_HandSoldering, F.Cu at (93.9, 53.6)
- added C5: 0.1uF, Capacitors_SMD:C_0402, F.Cu at (94.5, 64.8)
- added C6: 0.1uF, Capacitors_SMD:C_0402, F.Cu at (99.1, 59.1)
- added C7: 104, Capacitors_SMD:C_0603_HandSoldering, F.Cu at (115.7, 32.7)
- added C8: 104, Capacitors_SMD:C_0603_HandSoldering, F.Cu at (82.0, 35.2)
- added C9: 1uF, Capacitors_SMD:C_0402, F.Cu at (120.0, 38.0)
- added CON2: AVR-JTAG-10, Pin_Headers:Pin_Header_Straight_2x05, F.Cu at (90.7, 17.4)
- added Cff1: 33nF, Capacitors_SMD:C_0603_HandSoldering, F.Cu at (171.5, 10.1)
- added D1: LED_TX, LEDs:LED_0805, F.Cu at (84.5, 66.0)
- added D2: DIODESCH, Diodes_SMD:DO-214AB, F.Cu at (174.7, 1.51)
- added D3: LED_RX, LEDs:LED-8MM, F.Cu at (70.5, 50.9)
- added IC1: ATMEGA1280-A, Housings_QFP:TQFP-100_14x14mm_Pitch0.5mm, F.Cu at (147.3, 63.5)
- added JP1: JUMPER, Connect:PINHEAD1-2, F.Cu at (110.5, 34.7)
- added LM2596: LM2596, TO_SOT_Packages_SMD:TO-263-5Lead, F.Cu at (153.1, 2.07)
- added P1: CONN_02X20, Connect:IDC_Header_Straight_40pins, F.Cu at (176.5, 40.6)
- added P2: USB_OTG, Connect:USB_Micro-B, F.Cu at (81.7, 48.8)
- added R1: 220-470, Resistors_SMD:R_0805_HandSoldering, F.Cu at (80.6, 57.8)
- added R10: 150, Resistors_SMD:R_0402, F.Cu at (144.3, 15.8)
- added R11: 150, Resistors_SMD:R_0402, F.Cu at (141.0, 10.1)
- added R12: 470, Resistors_SMD:R_0805_HandSoldering, F.Cu at (96.6, 47.5)
- added R13: 470, Resistors_SMD:R_0805_HandSoldering, F.Cu at (79.0, 64.1)
- added R2: 220K, Resistors_SMD:R_0805_HandSoldering, F.Cu at (87.0, 60.1)
- added R3: 27, Resistors_SMD:R_0402, F.Cu at (90.9, 59.8)
- added R4: 27, Resistors_SMD:R_0402, F.Cu at (104.7, 47.2)
- added R5: 1.5K, Resistors_SMD:R_0402, F.Cu at (97.9, 53.5)
- added R6: R1, Resistors_SMD:R_0402, F.Cu at (138.0, 10.1)
- added R7: 220-470, Resistors_SMD:R_0805_HandSoldering, F.Cu at (90.3, 47.5)
- added R8: 220K, Resistors_SMD:R_0805_HandSoldering, F.Cu at (89.1, 53.8)
- added R9: 150, Resistors_SMD:R_0402, F.Cu at (144.4, 10.1)
- added U5: CONN3, Connect:Wafer_Vertical10x5.8x7RM2.5-3, F.Cu at (99.2, 34.6)
- added U6: WS2812, Connectors_Molex:Connector_Microfit3_Header_02x03_Straight_43045-0628, F.Cu at (137.8, 23.7)
- added U7: WS2812, Connectors_Molex:Connector_Microfit3_Header_02x03_Straight_43045-0628, F.Cu at (122.4, 23.7)
- added U8: WS2812, Connectors_Molex:Connector_Microfit3_Header_02x03_Straight_43045-0628, F.Cu at (106.9, 23.7)
- added U9: CONN3, Connect:Wafer_Vertical10x5.8x7RM2.5-3, F.Cu at (88.1, 34.6)
- added X1: CRYSTAL, Crystals:Crystal_FOX-FE_SMD, F.Cu at (141.2, 1.12)
- added Y1: CRYSTAL, Crystals:Crystal_FOX-FE_SMD, F.Cu at (71.8, 62.3)
- moved CON1 109.4 mm to (131.7, 2.42)
- moved C1 99.2 mm to (153.6, 10.5)
Connections:
- C1 pad 1: /PULSE -> /Vcc
- CON1 pad 1: /Sheet56DEE0DD/MOSI -> /Sheet56DEE0DD/CS
- CON1 pad 9: /Sheet56DEE0DD/MISO -> /Sheet56DEE0DD/Dout
Routing:
- net /Sheet56DEE0DD/D2: track 0.00 -> 28.6 mm
- net /Sheet56DEE0DD/A12: track 0.00 -> 26.0 mm

Commit message: Небольшие изменения в Pcbnew
Parts:
- moved D2 153.4 mm to (90.2, 129.5), turned to 90 degrees
- moved Cff1 148.9 mm to (105.4, 143.5)
- moved C2 148.5 mm to (110.5, 151.1)
- moved C1 137.3 mm to (119.4, 143.5), turned to 0 degrees
- moved LM2596 135.7 mm to (106.7, 129.5)
- moved CON1 128.8 mm to (142.2, 130.8)
- moved X1 120.6 mm to (157.5, 120.7)
- moved R11 68.1 mm to (151.1, 77.5)
- moved JP1 63.8 mm to (151.1, 83.8)
- moved C19 60.6 mm to (66.0, 96.5), turned to 90 degrees
- moved C5 52.1 mm to (96.5, 116.8)
- moved Y1 41.9 mm to (71.1, 104.1), turned to 90 degrees
- moved C12 41.0 mm to (131.6, 71.9)
- moved C17 41.0 mm to (119.4, 86.4)
- moved C22 41.0 mm to (85.1, 74.5)
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