File: Pulse_Module.kicad_pcb (KiCad board)
At the start: 2 copper layers, 61 parts, among them CON1 AVR-ISP-10, CON2 AVR-JTAG-10, CON3 BARREL_JACK, IC1 ATMEGA1280-A, P1 CONN_02X20, P2 USB_OTG, P3 CONN_01X03, P4 CONN_01X03, SW1 SW_PUSH, U1 74HCT541_PWR, U2 PL2303, U6 WS2812, U7 WS2812, U8 WS2812, X1 CRYSTAL, Y1 CRYSTAL

Commit message: LM2596
Parts:
- moved C2 3.84 mm to (115.1, 143.5)
- moved C1 1.27 mm to (114.0, 136.1)
- moved D2 0.76 mm to (115.6, 124.0)
Routing:
- net /Vcc: track 47.2 -> 42.5 mm
- net Net-(D2-Pad2): track 27.0 -> 26.2 mm
Changed lines of the file:
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@@
   (general
     (links 193)
-    (no_connects 153)
-    (area 0 0 0 0)
+    (no_connects 152)
+    (area 94.57552 58.157 275.511001 150.247)
     (thickness 1.6)
     (drawings 0)
-    (tracks 167)
+    (tracks 166)
     (zones 0)
     (modules 61)
@@
   )
   (module Diodes_SMD:DO-214AB (layer F.Cu)
-    (at 114.808 123.952 270)
+    (at 115.57 123.952 270)
     (descr "Jedec DO-214AB diode package. Designed according to Fairchild SS32 datasheet.")
     (tags "DO-214AB diode")
@@
   )
   (module Capacitors_SMD:C_0805 (layer F.Cu)
-    (at 111.252 144.018 180)
+    (at 115.062 143.51 180)
     (descr "Capacitor SMD 0805, reflow soldering, AVX (see smccp.pdf)")
     (tags "capacitor 0805")
@@
   )
   (module Capacitors_ThroughHole:C_Radial_D7.5_L11.2_P2.5 (layer F.Cu)
-    (at 112.776 136.144 180)
+    (at 114.046 136.144 180)
     (descr "Radial Electrolytic Capacitor Diameter 7.5mm x Length 11.2mm, Pitch 2.5mm")
     (tags "Electrolytic Capacitor")
@@
   (segment (start 200.82506 82.39506) (end 201.168 82.738) (width 0.25) (layer F.Cu) (net 2))
   (segment (start 164.004 106.624) (end 164.536 106.624) (width 0.25) (layer F.Cu) (net 5) (status 30))
-  (segment (start 130.69748 131.85548) (end 130.81 131.74296) (width 0.6) (layer F.Cu) (net 6))
-  (segment (start 130.81 131.74296) (end 130.81 128.762) (width 0.6) (layer F.Cu) (net 6))
-  (segment (start 116.69852 143.44142) (end 116.12194 144.018) (width 0.6) (layer F.Cu) (net 6))
-  (segment (start 116.12194 144.018) (end 112.252 144.018) (width 0.6) (layer F.Cu) (net 6))
-  (segment (start 123.698 143.44142) (end 116.69852 143.44142) (width 1) (layer F.Cu) (net 6))
-  (segment (start 116.69852 143.44142) (end 112.776 139.5189) (width 1) (layer F.Cu) (net 6))
-  (segment (start 112.776 139.5189) (end 112.776 136.144) (width 1) (layer F.Cu) (net 6))
+  (segment (start 130.69748 131.85548) (end 130.81 131.74296) (width 1) (layer F.Cu) (net 6))
+  (segment (start 130.81 131.74296) (end 130.81 128.762) (width 1) (layer F.Cu) (net 6))
+  (segment (start 123.698 143.44142) (end 126.94793 143.44142) (width 1) (layer F.Cu) (net 6))
+  (segment (start 126.94793 143.44142) (end 130.69748 139.69187) (width 1) (layer F.Cu) (net 6))
+  (segment (start 130.69748 139.69187) (end 130.69748 131.85548) (width 1) (layer F.Cu) (net 6))
+  (segment (start 116.062 143.51) (end 123.62942 143.51) (width 1) (layer F.Cu) (net 6))
+  (segment (start 123.62942 143.51) (end 123.698 143.44142) (width 1) (layer F.Cu) (net 6))
+  (segment (start 114.046 136.144) (end 114.046 141.494) (width 1) (layer F.Cu) (net 6))
+  (segment (start 114.046 141.494) (end 116.062 143.51) (width 1) (layer F.Cu) (net 6))
   (segment (start 127 128.458) (end 127.3 128.458) (width 1) (layer F.Cu) (net 6))
   (segment (start 127.3 128.458) (end 130.69748 131.85548) (width 1) (layer F.Cu) (net 6))
-  (segment (start 130.69748 131.85548) (end 130.69748 139.69187) (width 1) (layer F.Cu) (net 6))
-  (segment (start 130.69748 139.69187) (end 126.94793 143.44142) (width 1) (layer F.Cu) (net 6))
-  (segment (start 126.94793 143.44142) (end 123.698 143.44142) (width 1) (layer F.Cu) (net 6))
   (segment (start 122.49658 142.24) (end 123.698 143.44142) (width 1) (layer F.Cu) (net 6))
-  (segment (start 112.252 144.018) (end 112.252 144.288) (width 1) (layer F.Cu) (net 6) (status 30))
+  (segment (start 116.062 143.51) (end 116.062 143.78) (width 1) (layer F.Cu) (net 6) (status 30))
   (segment (start 136.652 94.742) (end 136.951999 94.442001) (width 0.4) (layer F.Cu) (net 12))
   (segment (start 136.951999 94.442001) (end 137.443999 94.442001) (width 0.4) (layer F.Cu) (net 12))
@@
   (segment (start 123.522 122.682) (end 123.209999 122.994001) (width 1) (layer F.Cu) (net 28))
   (segment (start 123.209999 122.994001) (end 123.209999 125.727999) (width 1) (layer F.Cu) (net 28))
-  (segment (start 117.856 128.27) (end 115.526 128.27) (width 1) (layer F.Cu) (net 28))
-  (segment (start 115.526 128.27) (end 114.808 127.552) (width 1) (layer F.Cu) (net 28))
+  (segment (start 117.856 128.27) (end 116.288 128.27) (width 1) (layer F.Cu) (net 28) (status 20))
+  (segment (start 116.288 128.27) (end 115.57 127.552) (width 1) (layer F.Cu) (net 28) (status 30))
   (segment (start 118.364 128.778) (end 117.856 128.27) (width 1) (layer B.Cu) (net 28))
   (via (at 117.856 128.27) (size 0.6) (drill 0.4) (layers F.Cu B.Cu) (net 28))
@@
   (via (at 122.428 130.048) (size 0.6) (drill 0.4) (layers F.Cu B.Cu) (net 28))
   (segment (start 123.698 134.94258) (end 126.94793 134.94258) (width 0.4) (layer F.Cu) (net 28) (status 30))
-  (segment (start 115.614 126.746) (end 114.808 127.552) (width 0.4) (layer F.Cu) (net 28) (status 30))
+  (segment (start 116.376 126.746) (end 115.57 127.552) (width 0.4) (layer F.Cu) (net 28) (status 30))
   (segment (start 175.204 110.824) (end 175.204 110.942) (width 0.25) (layer F.Cu) (net 57) (status 30))
   (segment (start 101.6 125.62586) (end 101.6 123.698) (width 1) (layer F.Cu) (net 97))

Commit message: исправлена LM2596
Parts:
- JP2: value JUMPER -> JUMPER3; footprint Connect:PINHEAD1-2 -> Connect:PINHEAD1-3
- moved CON1 62.6 mm to (129.5, 82.0), turned to 90 degrees
- moved Cff1 21.7 mm to (109.5, 123.7)
- moved C1 14.1 mm to (125.7, 128.3), turned to 270 degrees
- moved L1 13.3 mm to (136.7, 136.1)
- moved R10 13.0 mm to (127.3, 90.7)
- moved R14 12.9 mm to (114.6, 124.2), turned to 180 degrees
- moved LM2596 12.3 mm to (114.8, 129.3), turned to 270 degrees
- moved C2 12.3 mm to (126.7, 139.7)
- moved Y1 7.73 mm to (121.2, 85.3), turned to 180 degrees
- moved JP2 7.41 mm to (127.5, 118.4)
- moved D2 7.08 mm to (117.3, 117.1), turned to 0 degrees
- moved R15 6.49 mm to (118.9, 124.2), turned to 180 degrees
- moved P3 5.39 mm to (164.8, 133.3), turned to 270 degrees
- moved P4 5.33 mm to (151.4, 133.3), turned to 270 degrees
- moved P2 4.02 mm to (102.9, 90.9)
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Connections:
- JP2 pad 1: /Sheet56D88A8D/FB -> Net-(JP2-Pad1)
- R15 pad 1: /Sheet56D88A8D/FB -> Net-(JP2-Pad1)
Routing:
- net +5V: track 242.8 -> 166.9 mm
- net Net-(D2-Pad2): track 26.2 -> 43.1 mm, vias 3 -> 2
- net /Sheet56D88A8D/Vin: track 33.1 -> 20.0 mm, vias 0 -> 2
- net Net-(JP2-Pad1): track 0.00 -> 9.05 mm
- net /Sheet56D88A8D/FB: track 21.9 -> 13.6 mm
- net Net-(JP2-Pad2): track 7.98 -> 14.0 mm
- net /Vcc: track 42.5 -> 47.5 mm, vias 0 -> 4
- net +3V3: track 34.4 -> 36.6 mm

Commit message: Небольшие изменения
Connections:
- JP2 pad 3: Net-(JP2-Pad3) -> /Sheet56D88A8D/FB
Changed lines of the file:
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@@
 (kicad_pcb (version 4) (host pcbnew 4.0.2+dfsg1-2~bpo8+1-stable)
   (general
-    (links 192)
-    (no_connects 157)
+    (links 193)
+    (no_connects 156)
     (area 0 0 0 0)
     (thickness 1.6)
@@
     (zones 0)
     (modules 61)
-    (nets 148)
+    (nets 147)
   )
   (page A4)
@@
   )
   (setup
-    (last_trace_width 1)
+    (last_trace_width 0.25)
     (user_trace_width 0.3)
     (user_trace_width 0.4)
@@
   (net 145 "Net-(JP2-Pad2)")
   (net 146 "Net-(JP2-Pad1)")
-  (net 147 "Net-(JP2-Pad3)")
   (net_class Default "This is the default net class."
     (clearance 0.1)
@@
     (add_net "Net-(JP2-Pad1)")
     (add_net "Net-(JP2-Pad2)")
-    (add_net "Net-(JP2-Pad3)")
     (add_net "Net-(P1-Pad19)")
     (add_net "Net-(P2-Pad2)")
@@
       (net 145 "Net-(JP2-Pad2)"))
     (pad 3 thru_hole oval (at 2.54 0 90) (size 1.50622 3.01498) (drill 0.99822) (layers *.Cu *.Mask)
-      (net 147 "Net-(JP2-Pad3)"))
+      (net 16 /Sheet56D88A8D/FB))
   )
   (segment (start 178.139999 96.394999) (end 180.160001 96.394999) (width 0.25) (layer F.Cu) (net 0))
