File: ATmega1280.sch (KiCad schematic (older format))
At the start: 10 parts, among them CON1 AVR-ISP-10, IC1 ATMEGA1280-A, X1 CRYSTAL

Commit message: Добавление 40пинового разъёма и UART
Parts:
- added C?: 0.8, symbol C
- added JP?: JUMPER, symbol JUMPER
- added P?: CONN_02X20, symbol CONN_02X20
- added SW?: SW_PUSH, symbol SW_PUSH
- added U?: 74HCT541_PWR, symbol 74HCT541_PWR
- C: value C1 -> 1uF
- C? (x3): value C -> 100nF
Connections:
- net labels added: A0, A1, A10, A11, A12, A13, A14, A15, A16, A2, A3, A4, A5, A6, A7, A8, A9, ALE, CE, CLK, CS, CTS, D0, D1, D2, D3, D4, D5, D6, D7, Dout, I/O, RD, RTS, RXD, TXD, VCC, Vcc, WR
- wire segments 43 -> 64
- no-connect marks 1 -> 3
Other:
- moved on the sheet: C?, CON1

Commit message: Исправлено согласно комментариям
Parts:
- removed C?: 0.8, symbol C
- C10, C11, C12: renamed from C?; value 100nF -> 0.1uF
- gave numbers to parts that had none: 4
- renumbered C to C9, R to R6
Connections:
- net labels removed: CTS, RTS
- wire segments 64 -> 67
Changed lines of the file:
@@
 Sheet 3 4
 Title ""
-Date "7 apr 2016"
+Date "12 apr 2016"
 Rev ""
 Comp ""
@@
 $EndComp
 $Comp
-L +5V #PWR?
+L +5V #PWR5
 U 1 1 56E703CC
 P 3500 900
-F 0 "#PWR?" H 3500 750 50  0001 C CNN
+F 0 "#PWR5" H 3500 750 50  0001 C CNN
 F 1 "+5V" H 3500 1040 50  0000 C CNN
 F 2 "" H 3500 900 50  0000 C CNN
@@
 $EndComp
 $Comp
-L R R
+L R R6
 U 1 1 56E703F2
 P 3150 1350
-F 0 "R" V 3230 1350 50  0000 C CNN
+F 0 "R6" V 3230 1350 50  0000 C CNN
 F 1 "R1" V 3150 1350 50  0000 C CNN
 F 2 "" V 3080 1350 50  0000 C CNN
@@
 $EndComp
 $Comp
-L GND #PWR?
+L GND #PWR6
 U 1 1 56E704E1
 P 4450 7500
-F 0 "#PWR?" H 4450 7250 50  0001 C CNN
+F 0 "#PWR6" H 4450 7250 50  0001 C CNN
 F 1 "GND" H 4450 7350 50  0000 C CNN
 F 2 "" H 4450 7500 50  0000 C CNN
@@
 $EndComp
 $Comp
-L C C
+L C C9
 U 1 1 56E7056A
 P 2900 7300
-F 0 "C" H 2925 7400 50  0000 L CNN
+F 0 "C9" H 2925 7400 50  0000 L CNN
 F 1 "1uF" H 2925 7200 50  0000 L CNN
 F 2 "" H 2938 7150 50  0000 C CNN
@@
 $EndComp
 $Comp
-L GND #PWR?
+L GND #PWR4
 U 1 1 56E707E0
 P 2650 3550
-F 0 "#PWR?" H 2650 3300 50  0001 C CNN
+F 0 "#PWR4" H 2650 3300 50  0001 C CNN
 F 1 "GND" H 2650 3400 50  0000 C CNN
 F 2 "" H 2650 3550 50  0000 C CNN
@@
 $EndComp
 $Comp
-L C C?
+L C C10
 U 1 1 56E70D95
 P 9800 3100
-F 0 "C?" H 9825 3200 50  0000 L CNN
-F 1 "100nF" H 9825 3000 50  0000 L CNN
+F 0 "C10" H 9825 3200 50  0000 L CNN
+F 1 "0.1uF" H 9825 3000 50  0000 L CNN
 F 2 "" H 9838 2950 50  0000 C CNN
 F 3 "" H 9800 3100 50  0000 C CNN
@@
 $EndComp
 $Comp
-L C C?
+L C C11
 U 1 1 56E70DB0
 P 10150 3100
-F 0 "C?" H 10175 3200 50  0000 L CNN
-F 1 "100nF" H 10175 3000 50  0000 L CNN
+F 0 "C11" H 10175 3200 50  0000 L CNN
+F 1 "0.1uF" H 10175 3000 50  0000 L CNN
 F 2 "" H 10188 2950 50  0000 C CNN
 F 3 "" H 10150 3100 50  0000 C CNN
@@
 $EndComp
 $Comp
-L C C?
+L C C12
 U 1 1 56E70DBF
 P 10500 3100
-F 0 "C?" H 10525 3200 50  0000 L CNN
-F 1 "100nF" H 10525 3000 50  0000 L CNN
+F 0 "C12" H 10525 3200 50  0000 L CNN
+F 1 "0.1uF" H 10525 3000 50  0000 L CNN
 F 2 "" H 10538 2950 50  0000 C CNN
 F 3 "" H 10500 3100 50  0000 C CNN
@@
 $EndComp
 $Comp
-L GND #PWR?
+L GND #PWR11
 U 1 1 56E70DCE
-P 9850 3400
-F 0 "#PWR?" H 9850 3150 50  0001 C CNN
-F 1 "GND" H 9850 3250 50  0000 C CNN
-F 2 "" H 9850 3400 50  0000 C CNN
-F 3 "" H 9850 3400 50  0000 C CNN
-	1    9850 3400
+P 10150 3600
+F 0 "#PWR11" H 10150 3350 50  0001 C CNN
+F 1 "GND" H 10150 3450 50  0000 C CNN
+F 2 "" H 10150 3600 50  0000 C CNN
+F 3 "" H 10150 3600 50  0000 C CNN
+	1    10150 3600
 	1    0    0    -1
 $EndComp
@@
 MISO
 $Comp
-L GND #PWR?
+L GND #PWR13
 U 1 1 56E711C0
 P 10350 1700
-F 0 "#PWR?" H 10350 1450 50  0001 C CNN
+F 0 "#PWR13" H 10350 1450 50  0001 C CNN
 F 1 "GND" H 10350 1550 50  0000 C CNN
 F 2 "" H 10350 1700 50  0000 C CNN
@@
 RESET
 $Comp
-L +5V #PWR?
+L +5V #PWR12
 U 1 1 56E711D2
 P 10350 800
-F 0 "#PWR?" H 10350 650 50  0001 C CNN
+F 0 "#PWR12" H 10350 650 50  0001 C CNN
 F 1 "+5V" H 10350 940 50  0000 C CNN
 F 2 "" H 10350 800 50  0000 C CNN
@@
 NoConn ~ 9400 1200
 $Comp
-L JUMPER JP?
+L JUMPER JP1
 U 1 1 56F2E87D
 P 2850 1100
-F 0 "JP?" H 2850 1250 50  0000 C CNN
+F 0 "JP1" H 2850 1250 50  0000 C CNN
 F 1 "JUMPER" H 2850 1020 50  0000 C CNN
 F 2 "" H 2850 1100 50  0000 C CNN
@@
 Vcc
 Wire Wire Line
-	9800 3350 9800 3200
+	9800 3350 9800 3250
 Wire Wire Line
 	10500 3350 10500 3250
@@
 	10150 3250 10150 3600
 $Comp
-L +5V #PWR?
+L +5V #PWR10
 U 1 1 56F4EFCF
 P 10150 2500
-F 0 "#PWR?" H 10150 2350 50  0001 C CNN
+F 0 "#PWR10" H 10150 2350 50  0001 C CNN
 F 1 "+5V" H 10150 2640 50  0000 C CNN
 F 2 "" H 10150 2500 50  0000 C CNN
@@
 	9800 3350 10500 3350
 $Comp
-L SW_PUSH SW?
+L SW_PUSH SW1
 U 1 1 56F4F0F3
 P 2150 1750
-F 0 "SW?" H 2300 1860 50  0000 C CNN
+F 0 "SW1" H 2300 1860 50  0000 C CNN
 F 1 "SW_PUSH" H 2150 1670 50  0000 C CNN
 F 2 "" H 2150 1750 50  0000 C CNN
@@
 $EndComp
 $Comp
-L GND #PWR?
+L GND #PWR3
 U 1 1 56F4F102
 P 1450 2000
-F 0 "#PWR?" H 1450 1750 50  0001 C CNN
+F 0 "#PWR3" H 1450 1750 50  0001 C CNN
 F 1 "GND" H 1450 1850 50  0000 C CNN
 F 2 "" H 1450 2000 50  0000 C CNN
@@
 	1450 1750 1850 1750
 Wire Wire Line
-	3150 1100 4300 1100
+	3150 1100 4600 1100
 $Sheet
 S 8100 4550 950  550
@@
 $EndSheet
 $Comp
-L GND #PWR?
-U 1 1 570520C0
-P 9850 3400
-F 0 "#PWR?" H 9850 3150 50  0001 C CNN
-F 1 "GND" H 9850 3250 50  0000 C CNN
-F 2 "" H 9850 3400 50  0000 C CNN
-F 3 "" H 9850 3400 50  0000 C CNN
-	1    9850 3400
-	1    0    0    -1
-$EndComp
-$Comp
-L CONN_02X20 P?
+L CONN_02X20 P1
 U 1 1 5706199C
 P 9050 3000
-F 0 "P?" H 9050 4050 50  0000 C CNN
+F 0 "P1" H 9050 4050 50  0000 C CNN
 F 1 "CONN_02X20" V 9050 3000 50  0000 C CNN
 F 2 "" H 9050 2050 50  0000 C CNN
@@
 Text Label 3150 4550 2    60   ~ 0
 TXD
-Text HLabel 9050 4650 0    60   Input ~ 0
-CTS
-Text HLabel 9050 4800 0    60   Input ~ 0
-RTS
-$Comp
-L 74HCT541_PWR U?
+$Comp
+L 74HCT541_PWR U1
 U 1 1 5706A061
 P 7550 2250
-F 0 "U?" H 7650 2900 50  0000 L CNN
+F 0 "U1" H 7650 2900 50  0000 L CNN
 F 1 "74HCT541_PWR" H 7600 1600 50  0000 L CNN
 F 2 "" H 7550 2250 50  0000 C CNN
@@
 	7550 3000 7550 3150
 $Comp
-L GND #PWR?
+L GND #PWR8
 U 1 1 5706A0E3
 P 7550 3150
-F 0 "#PWR?" H 7550 2900 50  0001 C CNN
+F 0 "#PWR8" H 7550 2900 50  0001 C CNN
 F 1 "GND" H 7550 3000 50  0000 C CNN
 F 2 "" H 7550 3150 50  0000 C CNN
@@
 $EndComp
 $Comp
-L C C?
-U 1 1 5706A0F2
-P 7550 1250
-F 0 "C?" H 7575 1350 50  0000 L CNN
-F 1 "0.8" H 7575 1150 50  0000 L CNN
-F 2 "" H 7588 1100 50  0000 C CNN
-F 3 "" H 7550 1250 50  0000 C CNN
-	1    7550 1250
-	1    0    0    -1
-$EndComp
-$Comp
-L VCC #PWR?
+L VCC #PWR7
 U 1 1 5706A106
-P 7550 1000
-F 0 "#PWR?" H 7550 850 50  0001 C CNN
-F 1 "VCC" H 7550 1150 50  0000 C CNN
-F 2 "" H 7550 1000 50  0000 C CNN
-F 3 "" H 7550 1000 50  0000 C CNN
-	1    7550 1000
-	1    0    0    -1
-$EndComp
-Wire Wire Line
-	7550 1000 7550 1100
-Wire Wire Line
-	7550 1400 7550 1500
+P 7550 1300
+F 0 "#PWR7" H 7550 1150 50  0001 C CNN
+F 1 "VCC" H 7550 1450 50  0000 C CNN
+F 2 "" H 7550 1300 50  0000 C CNN
+F 3 "" H 7550 1300 50  0000 C CNN
+	1    7550 1300
+	1    0    0    -1
+$EndComp
+Wire Wire Line
+	7550 1300 7550 1500
 Text Label 8800 2050 2    60   ~ 0
 D0
@@
 Connection ~ 9500 3950
 $Comp
-L GND #PWR?
+L GND #PWR9
 U 1 1 5706A2FA
 P 9500 4050
-F 0 "#PWR?" H 9500 3800 50  0001 C CNN
+F 0 "#PWR9" H 9500 3800 50  0001 C CNN
 F 1 "GND" H 9500 3900 50  0000 C CNN
 F 2 "" H 9500 4050 50  0000 C CNN
@@
 Wire Wire Line
 	5750 2450 6850 2450
-Text Label 5750 1750 0    60   ~ 0
+Text Label 5950 1750 0    60   ~ 0
 D0
-Text Label 5750 1850 0    60   ~ 0
+Text Label 5950 1850 0    60   ~ 0
 D1
-Text Label 5750 1950 0    60   ~ 0
+Text Label 5950 1950 0    60   ~ 0
 D2
 Text Label 5750 2050 0    60   ~ 0
@@
 Text Label 3150 6350 2    60   ~ 0
 RD
+Wire Wire Line
+	4600 1100 4600 1450
+Text HLabel 9050 4950 0    60   Input ~ 0
+RESET
+Text Label 9450 4950 2    60   ~ 0
+RESET
+Wire Wire Line
+	9050 4950 9450 4950
+Wire Wire Line
+	8100 4650 7800 4650
+Wire Wire Line
+	8100 4800 7800 4800
+Text Label 7800 4650 0    60   ~ 0
+RXD
+Text Label 7800 4800 0    60   ~ 0
+TXD
 $EndSCHEMATC

Commit message: Аннотированные элементы
Parts:
- renumbered C2 to C21, C1 to C22
Connections:
- wire segments 67 -> 69
- no-connect marks 3 -> 65
Changed lines of the file:
@@
 Sheet 3 4
 Title ""
-Date "12 apr 2016"
+Date "14 apr 2016"
 Rev ""
 Comp ""
@@
 $EndComp
 $Comp
-L +5V #PWR5
+L +5V #PWR03
 U 1 1 56E703CC
 P 3500 900
-F 0 "#PWR5" H 3500 750 50  0001 C CNN
+F 0 "#PWR03" H 3500 750 50  0001 C CNN
 F 1 "+5V" H 3500 1040 50  0000 C CNN
 F 2 "" H 3500 900 50  0000 C CNN
@@
 $EndComp
 $Comp
-L GND #PWR6
+L GND #PWR04
 U 1 1 56E704E1
 P 4450 7500
-F 0 "#PWR6" H 4450 7250 50  0001 C CNN
+F 0 "#PWR04" H 4450 7250 50  0001 C CNN
 F 1 "GND" H 4450 7350 50  0000 C CNN
 F 2 "" H 4450 7500 50  0000 C CNN
@@
 $EndComp
 $Comp
-L C C1
+L C C22
 U 1 1 56E70771
 P 1950 3100
-F 0 "C1" H 1975 3200 50  0000 L CNN
+F 0 "C22" H 1975 3200 50  0000 L CNN
 F 1 "27pF" H 1975 3000 50  0000 L CNN
 F 2 "" H 1988 2950 50  0000 C CNN
@@
 $EndComp
 $Comp
-L C C2
+L C C21
 U 1 1 56E70780
 P 2650 3100
-F 0 "C2" H 2675 3200 50  0000 L CNN
+F 0 "C21" H 2675 3200 50  0000 L CNN
 F 1 "27pF" H 2675 3000 50  0000 L CNN
 F 2 "" H 2688 2950 50  0000 C CNN
@@
 $EndComp
 $Comp
-L GND #PWR4
+L GND #PWR05
 U 1 1 56E707E0
 P 2650 3550
-F 0 "#PWR4" H 2650 3300 50  0001 C CNN
+F 0 "#PWR05" H 2650 3300 50  0001 C CNN
 F 1 "GND" H 2650 3400 50  0000 C CNN
 F 2 "" H 2650 3550 50  0000 C CNN
@@
 $EndComp
 $Comp
-L GND #PWR11
+L GND #PWR06
 U 1 1 56E70DCE
 P 10150 3600
-F 0 "#PWR11" H 10150 3350 50  0001 C CNN
+F 0 "#PWR06" H 10150 3350 50  0001 C CNN
 F 1 "GND" H 10150 3450 50  0000 C CNN
 F 2 "" H 10150 3600 50  0000 C CNN
@@
 MISO
 $Comp
-L GND #PWR13
+L GND #PWR07
 U 1 1 56E711C0
 P 10350 1700
-F 0 "#PWR13" H 10350 1450 50  0001 C CNN
+F 0 "#PWR07" H 10350 1450 50  0001 C CNN
 F 1 "GND" H 10350 1550 50  0000 C CNN
 F 2 "" H 10350 1700 50  0000 C CNN
@@
 RESET
 $Comp
-L +5V #PWR12
+L +5V #PWR08
 U 1 1 56E711D2
 P 10350 800
-F 0 "#PWR12" H 10350 650 50  0001 C CNN
+F 0 "#PWR08" H 10350 650 50  0001 C CNN
 F 1 "+5V" H 10350 940 50  0000 C CNN
 F 2 "" H 10350 800 50  0000 C CNN
@@
 	10150 3250 10150 3600
 $Comp
-L +5V #PWR10
+L +5V #PWR09
 U 1 1 56F4EFCF
 P 10150 2500
-F 0 "#PWR10" H 10150 2350 50  0001 C CNN
+F 0 "#PWR09" H 10150 2350 50  0001 C CNN
 F 1 "+5V" H 10150 2640 50  0000 C CNN
 F 2 "" H 10150 2500 50  0000 C CNN
@@
 $EndComp
 $Comp
-L GND #PWR3
+L GND #PWR010
 U 1 1 56F4F102
 P 1450 2000
-F 0 "#PWR3" H 1450 1750 50  0001 C CNN
+F 0 "#PWR010" H 1450 1750 50  0001 C CNN
 F 1 "GND" H 1450 1850 50  0000 C CNN
 F 2 "" H 1450 2000 50  0000 C CNN
@@
 Text HLabel 8100 4800 2    60   Input ~ 0
 TXD
-Text Label 3150 4450 2    60   ~ 0
+Text Label 2800 4450 0    60   ~ 0
 RXD
-Text Label 3150 4550 2    60   ~ 0
+Text Label 2800 4550 0    60   ~ 0
 TXD
 $Comp
@@
 	7550 3000 7550 3150
 $Comp
-L GND #PWR8
+L GND #PWR011
 U 1 1 5706A0E3
 P 7550 3150
-F 0 "#PWR8" H 7550 2900 50  0001 C CNN
+F 0 "#PWR011" H 7550 2900 50  0001 C CNN
 F 1 "GND" H 7550 3000 50  0000 C CNN
 F 2 "" H 7550 3150 50  0000 C CNN
@@
 $EndComp
 $Comp
-L VCC #PWR7
+L VCC #PWR012
 U 1 1 5706A106
 P 7550 1300
-F 0 "#PWR7" H 7550 1150 50  0001 C CNN
+F 0 "#PWR012" H 7550 1150 50  0001 C CNN
 F 1 "VCC" H 7550 1450 50  0000 C CNN
 F 2 "" H 7550 1300 50  0000 C CNN
@@
 Connection ~ 9500 3950
 $Comp
-L GND #PWR9
+L GND #PWR013
 U 1 1 5706A2FA
 P 9500 4050
-F 0 "#PWR9" H 9500 3800 50  0001 C CNN
+F 0 "#PWR013" H 9500 3800 50  0001 C CNN
 F 1 "GND" H 9500 3900 50  0000 C CNN
 F 2 "" H 9500 4050 50  0000 C CNN
@@
 Text Label 7800 4800 0    60   ~ 0
 TXD
+Wire Wire Line
+	3150 4450 2800 4450
+Wire Wire Line
+	3150 4550 2800 4550
+NoConn ~ 3150 2650
+NoConn ~ 3150 2750
+NoConn ~ 3150 2850
+NoConn ~ 3150 2950
+NoConn ~ 3150 3050
+NoConn ~ 3150 3150
+NoConn ~ 3150 3250
+NoConn ~ 3150 3350
+NoConn ~ 3150 3550
+NoConn ~ 3150 3650
+NoConn ~ 3150 3750
+NoConn ~ 3150 3850
+NoConn ~ 3150 3950
+NoConn ~ 3150 4050
+NoConn ~ 3150 4150
+NoConn ~ 3150 4250
+NoConn ~ 3150 4650
+NoConn ~ 3150 4750
+NoConn ~ 3150 4850
+NoConn ~ 3150 4950
+NoConn ~ 3150 5050
+NoConn ~ 3150 5150
+NoConn ~ 3150 5350
+NoConn ~ 3150 5450
+NoConn ~ 3150 5550
+NoConn ~ 3150 5650
+NoConn ~ 3150 5750
+NoConn ~ 3150 5850
+NoConn ~ 3150 5950
+NoConn ~ 3150 6050
+NoConn ~ 3150 6550
+NoConn ~ 3150 6650
+NoConn ~ 3150 6750
+NoConn ~ 5750 6950
+NoConn ~ 5750 6850
+NoConn ~ 5750 6750
+NoConn ~ 5750 6650
+NoConn ~ 5750 6550
+NoConn ~ 5750 6450
+NoConn ~ 5750 6350
+NoConn ~ 5750 6250
+NoConn ~ 5750 6050
+NoConn ~ 5750 5950
+NoConn ~ 5750 5850
+NoConn ~ 5750 5750
+NoConn ~ 5750 5650
+NoConn ~ 5750 5550
+NoConn ~ 5750 5450
+NoConn ~ 5750 5350
+NoConn ~ 5750 5150
+NoConn ~ 5750 5050
+NoConn ~ 5750 4950
+NoConn ~ 5750 4850
+NoConn ~ 5750 4750
+NoConn ~ 5750 4650
+NoConn ~ 5750 4550
+NoConn ~ 5750 4450
+NoConn ~ 5750 3350
+NoConn ~ 5750 3250
+NoConn ~ 5750 3150
+NoConn ~ 5750 3050
+NoConn ~ 5750 2650
 $EndSCHEMATC

Commit message: исправление ошибок
Parts:
- added U?: CONN3, symbol CONN3
Connections:
- net labels added: CE2, RXD0, RXD1, TXD0, TXD1
- wire segments 69 -> 75
- no-connect marks 65 -> 63
Changed lines of the file:
@@
 EESchema Schematic File Version 2
+LIBS:conn3
 LIBS:pl2303
 LIBS:power
@@
 Sheet 3 4
 Title ""
-Date "14 apr 2016"
+Date "20 apr 2016"
 Rev ""
 Comp ""
@@
 RXD
 Text HLabel 8100 4800 2    60   Input ~ 0
-TXD
-Text Label 2800 4450 0    60   ~ 0
-RXD
-Text Label 2800 4550 0    60   ~ 0
 TXD
 $Comp
@@
 $EndComp
 Text Label 9300 3750 0    60   ~ 0
-CE
+CE2
 Text Label 8250 2050 0    60   ~ 0
 A3
@@
 	8100 4800 7800 4800
 Text Label 7800 4650 0    60   ~ 0
-RXD
+RXD0
 Text Label 7800 4800 0    60   ~ 0
-TXD
-Wire Wire Line
-	3150 4450 2800 4450
-Wire Wire Line
-	3150 4550 2800 4550
+TXD0
 NoConn ~ 3150 2650
 NoConn ~ 3150 2750
@@
 NoConn ~ 5750 5650
 NoConn ~ 5750 5550
-NoConn ~ 5750 5450
-NoConn ~ 5750 5350
 NoConn ~ 5750 5150
 NoConn ~ 5750 5050
 NoConn ~ 5750 4950
 NoConn ~ 5750 4850
-NoConn ~ 5750 4750
-NoConn ~ 5750 4650
-NoConn ~ 5750 4550
 NoConn ~ 5750 4450
 NoConn ~ 5750 3350
@@
 NoConn ~ 5750 3050
 NoConn ~ 5750 2650
+Wire Wire Line
+	5750 5350 6000 5350
+Text Label 6000 5350 2    60   ~ 0
+RXD0
+Wire Wire Line
+	5750 5450 6000 5450
+Text Label 6000 5450 2    60   ~ 0
+TXD0
+NoConn ~ 5750 4550
+Wire Wire Line
+	5750 4650 6050 4650
+Wire Wire Line
+	5750 4750 6050 4750
+Text Label 6050 4650 2    60   ~ 0
+RXD1
+Text Label 6050 4750 2    60   ~ 0
+TXD1
+NoConn ~ 3150 4450
+NoConn ~ 3150 4550
+$Comp
+L CONN3 U?
+U 1 1 5717E35D
+P 7250 5400
+F 0 "U?" H 7600 4750 60  0000 C CNN
+F 1 "CONN3" H 7600 5150 60  0000 C CNN
+F 2 "" H 7250 5400 60  0000 C CNN
+F 3 "" H 7250 5400 60  0000 C CNN
+	1    7250 5400
+	1    0    0    -1
+$EndComp
+Wire Wire Line
+	8050 5600 8450 5600
+Wire Wire Line
+	8050 5700 8450 5700
+Wire Wire Line
+	8050 5800 8450 5800
+Wire Wire Line
+	8450 5800 8450 5900
+$Comp
+L GND #PWR?
+U 1 1 5717E47B
+P 8450 5900
+F 0 "#PWR?" H 8450 5650 50  0001 C CNN
+F 1 "GND" H 8450 5750 50  0000 C CNN
+F 2 "" H 8450 5900 50  0000 C CNN
+F 3 "" H 8450 5900 50  0000 C CNN
+	1    8450 5900
+	1    0    0    -1
+$EndComp
+Text Label 8450 5600 2    60   ~ 0
+RXD1
+Text Label 8450 5700 2    60   ~ 0
+TXD1
 $EndSCHEMATC

Commit message: Добавление WS2812, исправление всех замечаний
Parts:
- added C? (x3): 104, symbol C
- added R? (x3): 150, symbol R
- added U?: CONN3, symbol CONN3
- added U? (x3): WS2812, symbol WS2812
- CON1: footprint AVR-ISP-10 -> Pin_Headers:Pin_Header_Straight_2x05
- X1: symbol CRYSTAL -> Crystal
- gave numbers to parts that had none: 1
Connections:
- net labels added: 17, 21, 23, 25, 27, 34
- net labels removed: A16, I/O, VCC
- wire segments 75 -> 173
- no-connect marks 63 -> 59
