File: pl2303.sch (KiCad schematic (older format))
At the start: 57 parts

Commit message: Исправлено согласно комментариям
Parts:
- removed C1, C2, C? (x6): 10P, symbol C
- removed C? (x6): 0.1U, symbol C
- removed R5, R6: 4.7K, symbol R
- removed R? (x6): 220K, symbol R
- removed R? (x3): R, symbol R
- removed Y? (x4): CRYSTAL, symbol CRYSTAL
- added C14: 0.1uF, symbol C
- added C19, C20: C, symbol C
- added Y1: CRYSTAL, symbol CRYSTAL
- C4: value 0.1U -> C
- R1: value 220K -> 220-470
- gave numbers to parts that had none: 10
- renumbered FB to FB1, FB to FB2, FB to FB3, FB to FB4
Connections:
- net labels added: +3.3V, D+, D-, GND_3V3, RESET, VDD_3V3, VDD_PLL
- net labels removed: 13, 14, 15, 16, 17, 18, 19, 20, 21, 22, 23, 24, 25, 26, 27, 28, 4, 7, 8, CTS, RTS
- wire segments 103 -> 115
- no-connect marks 3 -> 11
Other:
- moved on the sheet: C3

Commit message: Аннотированные элементы
Parts:
- removed C5, C7: 0.1U, symbol C
- removed C6, C8: 10U, symbol C
- FB4: value C2 -> L2
Connections:
- wire segments 115 -> 94
Changed lines of the file:
@@
 Sheet 4 4
 Title ""
-Date "12 apr 2016"
+Date "13 apr 2016"
 Rev ""
 Comp ""
@@
 U 1 1 570525EF
 P 2550 3300
-F 0 "U2" H 2950 1550 60  0000 C CNN
+F 0 "U2" H 3250 1550 60  0000 C CNN
 F 1 "PL2303" H 2950 3050 60  0000 C CNN
 F 2 "" H 2550 3300 60  0000 C CNN
@@
 U 1 1 57052646
 P 2550 3300
-F 0 "U3" H 2950 1550 60  0000 C CNN
+F 0 "U3" H 2600 1550 60  0000 C CNN
 F 1 "PL2303" H 2950 3050 60  0000 C CNN
 F 2 "" H 2550 3300 60  0000 C CNN
@@
 U 1 1 570526B8
 P 2550 3300
-F 0 "U4" H 2950 1550 60  0000 C CNN
+F 0 "U4" H 3450 1350 60  0000 C CNN
 F 1 "PL2303" H 2950 3050 60  0000 C CNN
 F 2 "" H 2550 3300 60  0000 C CNN
@@
 $EndComp
 $Comp
-L C C5
-U 1 1 57052724
-P 7400 3850
-F 0 "C5" H 7425 3950 50  0000 L CNN
-F 1 "0.1U" H 7425 3750 50  0000 L CNN
-F 2 "" H 7438 3700 50  0000 C CNN
-F 3 "" H 7400 3850 50  0000 C CNN
-	1    7400 3850
-	1    0    0    -1
-$EndComp
-$Comp
-L C C6
-U 1 1 5705277E
-P 7850 3850
-F 0 "C6" H 7875 3950 50  0000 L CNN
-F 1 "10U" H 7875 3750 50  0000 L CNN
-F 2 "" H 7888 3700 50  0000 C CNN
-F 3 "" H 7850 3850 50  0000 C CNN
-	1    7850 3850
-	1    0    0    -1
-$EndComp
-$Comp
-L GND #PWR25
+L GND #PWR014
 U 1 1 5705278D
 P 8200 3600
-F 0 "#PWR25" H 8200 3350 50  0001 C CNN
+F 0 "#PWR014" H 8200 3350 50  0001 C CNN
 F 1 "GND" H 8200 3450 50  0000 C CNN
 F 2 "" H 8200 3600 50  0000 C CNN
@@
 $EndComp
 $Comp
-L C C7
-U 1 1 57052912
-P 6650 5300
-F 0 "C7" H 6675 5400 50  0000 L CNN
-F 1 "0.1U" H 6675 5200 50  0000 L CNN
-F 2 "" H 6688 5150 50  0000 C CNN
-F 3 "" H 6650 5300 50  0000 C CNN
-	1    6650 5300
-	1    0    0    -1
-$EndComp
-$Comp
-L C C8
-U 1 1 57052918
-P 7100 5300
-F 0 "C8" H 7125 5400 50  0000 L CNN
-F 1 "10U" H 7125 5200 50  0000 L CNN
-F 2 "" H 7138 5150 50  0000 C CNN
-F 3 "" H 7100 5300 50  0000 C CNN
-	1    7100 5300
-	1    0    0    -1
-$EndComp
-$Comp
 L C C15
 U 1 1 57052926
@@
 P 7900 5000
 F 0 "FB4" V 7850 5000 50  0000 C CNN
-F 1 "C2" V 8000 5000 50  0000 C CNN
+F 1 "L2" V 8000 5000 50  0000 C CNN
 F 2 "" H 7900 5000 50  0000 C CNN
 F 3 "" H 7900 5000 50  0000 C CNN
@@
 $EndComp
 $Comp
-L GND #PWR24
+L GND #PWR015
 U 1 1 57052951
 P 7350 5600
-F 0 "#PWR24" H 7350 5350 50  0001 C CNN
+F 0 "#PWR015" H 7350 5350 50  0001 C CNN
 F 1 "GND" H 7350 5450 50  0000 C CNN
 F 2 "" H 7350 5600 50  0000 C CNN
@@
 $EndComp
 $Comp
-L GND #PWR23
+L GND #PWR016
 U 1 1 570529E3
 P 7300 4700
-F 0 "#PWR23" H 7300 4450 50  0001 C CNN
+F 0 "#PWR016" H 7300 4450 50  0001 C CNN
 F 1 "GND" H 7300 4550 50  0000 C CNN
 F 2 "" H 7300 4700 50  0000 C CNN
@@
 $EndComp
 $Comp
-L GND #PWR16
+L GND #PWR017
 U 1 1 570570AA
 P 1300 5000
-F 0 "#PWR16" H 1300 4750 50  0001 C CNN
+F 0 "#PWR017" H 1300 4750 50  0001 C CNN
 F 1 "GND" H 1300 4850 50  0000 C CNN
 F 2 "" H 1300 5000 50  0000 C CNN
@@
 $EndComp
 $Comp
-L VDD #PWR15
+L VDD #PWR018
 U 1 1 570570B9
 P 1300 4450
-F 0 "#PWR15" H 1300 4300 50  0001 C CNN
+F 0 "#PWR018" H 1300 4300 50  0001 C CNN
 F 1 "VDD" H 1300 4600 50  0000 C CNN
 F 2 "" H 1300 4450 50  0000 C CNN
@@
 $EndComp
 $Comp
-L GND #PWR19
+L GND #PWR019
 U 1 1 570620C0
 P 2950 5500
-F 0 "#PWR19" H 2950 5250 50  0001 C CNN
+F 0 "#PWR019" H 2950 5250 50  0001 C CNN
 F 1 "GND" H 2950 5350 50  0000 C CNN
 F 2 "" H 2950 5500 50  0000 C CNN
@@
 $EndComp
 $Comp
-L VCC #PWR22
+L VCC #PWR020
 U 1 1 5706293A
 P 6350 4800
-F 0 "#PWR22" H 6350 4650 50  0001 C CNN
+F 0 "#PWR020" H 6350 4650 50  0001 C CNN
 F 1 "VCC" H 6350 4950 50  0000 C CNN
 F 2 "" H 6350 4800 50  0000 C CNN
@@
 $EndComp
 Wire Wire Line
-	7150 3550 7400 3550
-Wire Wire Line
-	7400 3550 7850 3550
-Wire Wire Line
-	7850 3550 8200 3550
+	7150 3550 8200 3550
 Wire Wire Line
 	7400 3550 7400 3700
@@
 Connection ~ 7850 3550
 Wire Wire Line
-	7150 4000 7400 4000
-Wire Wire Line
-	7400 4000 7850 4000
-Wire Wire Line
-	7850 4000 8600 4000
+	7150 4000 8600 4000
 Connection ~ 7400 4000
 Connection ~ 7850 4000
@@
 	6650 5450 6650 5600
 Wire Wire Line
-	6650 5600 7100 5600
-Wire Wire Line
-	7100 5600 7350 5600
+	6650 5600 7350 5600
 Wire Wire Line
 	7100 5600 7100 5450
 Connection ~ 7100 5600
 Wire Wire Line
-	6350 5000 6650 5000
-Wire Wire Line
-	6650 5000 7100 5000
-Wire Wire Line
-	7100 5000 7600 5000
+	6350 5000 7600 5000
 Wire Wire Line
 	8200 5000 8650 5000
@@
 	6900 6050 7350 6050
 Wire Wire Line
-	6900 6300 7100 6300
-Wire Wire Line
-	7100 6300 7350 6300
+	6900 6300 7350 6300
 Wire Wire Line
 	7100 6300 7100 6450
@@
 	3100 4950 3550 4950
 Wire Wire Line
-	4150 4150 4200 4150
-Wire Wire Line
-	4200 4150 4400 4150
+	4150 4150 4400 4150
 Wire Wire Line
 	3550 3900 4000 3900
@@
 	4000 3900 4000 4300
 Wire Wire Line
-	4000 4300 4050 4300
-Wire Wire Line
-	4050 4300 4400 4300
+	4000 4300 4400 4300
 Wire Wire Line
 	3950 4650 4050 4650
@@
 $EndComp
 $Comp
-L GND #PWR14
+L GND #PWR021
 U 1 1 570D14D2
 P 950 3800
-F 0 "#PWR14" H 950 3550 50  0001 C CNN
+F 0 "#PWR021" H 950 3550 50  0001 C CNN
 F 1 "GND" H 950 3650 50  0000 C CNN
 F 2 "" H 950 3800 50  0000 C CNN
@@
 	800  3300 600  3300
 Wire Wire Line
-	600  2900 600  3300
-Wire Wire Line
-	600  3300 600  3350
+	600  2900 600  3350
 Wire Wire Line
 	600  3650 600  3750
 Wire Wire Line
-	600  3750 950  3750
-Wire Wire Line
-	950  3750 1300 3750
+	600  3750 1300 3750
 Wire Wire Line
 	950  3750 950  3800
@@
 Connection ~ 950  3750
 Wire Wire Line
-	1300 3000 1300 3300
-Wire Wire Line
-	1300 3300 1300 3350
+	1300 3000 1300 3350
 Wire Wire Line
 	1300 3300 1100 3300
@@
 	2800 5350 2800 5450
 Wire Wire Line
-	2800 5450 2950 5450
-Wire Wire Line
-	2950 5450 3100 5450
+	2800 5450 3100 5450
 Wire Wire Line
 	2950 5450 2950 5500
@@
 	3550 2700 4100 2700
 Wire Wire Line
-	2450 4300 2450 4450
-Wire Wire Line
-	2450 4450 2450 4600
-Wire Wire Line
-	2450 4600 2450 4650
+	2450 4300 2450 4650
 Wire Wire Line
 	3550 3000 3700 3000
@@
 Connection ~ 2450 4450
 $Comp
-L GND #PWR18
+L GND #PWR022
 U 1 1 570D2EBB
 P 2450 5100
-F 0 "#PWR18" H 2450 4850 50  0001 C CNN
+F 0 "#PWR022" H 2450 4850 50  0001 C CNN
 F 1 "GND" H 2450 4950 50  0000 C CNN
 F 2 "" H 2450 5100 50  0000 C CNN
@@
 $EndComp
 Wire Wire Line
-	2450 4950 2450 5050
-Wire Wire Line
-	2450 5050 2450 5100
+	2450 4950 2450 5100
 $Comp
 L R R2
@@
 $EndComp
 $Comp
-L GND #PWR21
+L GND #PWR023
 U 1 1 570D2F71
 P 4850 3050
-F 0 "#PWR21" H 4850 2800 50  0001 C CNN
+F 0 "#PWR023" H 4850 2800 50  0001 C CNN
 F 1 "GND" H 4850 2900 50  0000 C CNN
 F 2 "" H 4850 3050 50  0000 C CNN
@@
 $EndComp
 $Comp
-L VDD #PWR20
+L VDD #PWR024
 U 1 1 570D309D
 P 4600 1700
-F 0 "#PWR20" H 4600 1550 50  0001 C CNN
+F 0 "#PWR024" H 4600 1550 50  0001 C CNN
 F 1 "VDD" H 4600 1850 50  0000 C CNN
 F 2 "" H 4600 1700 50  0000 C CNN
@@
 	4600 2800 4500 2800
 Wire Wire Line
-	4600 1700 4600 2200
-Wire Wire Line
-	4600 2200 4600 2800
+	4600 1700 4600 2800
 Wire Wire Line
 	2650 2300 2650 2200
 Wire Wire Line
-	2650 2200 4100 2200
-Wire Wire Line
-	4100 2200 4300 2200
-Wire Wire Line
-	4300 2200 4600 2200
+	2650 2200 4600 2200
 Wire Wire Line
 	4100 2700 4100 2200
@@
 	4300 1850 4850 1850
 Wire Wire Line
-	4850 1850 4850 2900
-Wire Wire Line
-	4850 2900 4850 3050
+	4850 1850 4850 3050
 Connection ~ 4850 2900
 Text Label 2750 2300 0    60   ~ 0
@@
 	8600 4000 8600 3250
 $Comp
-L +3.3V #PWR26
+L +3.3V #PWR025
 U 1 1 570D3933
 P 8600 3250
-F 0 "#PWR26" H 8600 3100 50  0001 C CNN
+F 0 "#PWR025" H 8600 3100 50  0001 C CNN
 F 1 "+3.3V" H 8600 3390 50  0000 C CNN
 F 2 "" H 8600 3250 50  0000 C CNN
@@
 GND_3V3
 $Comp
-L GND #PWR17
+L GND #PWR026
 U 1 1 570D3A89
 P 2350 4400
-F 0 "#PWR17" H 2350 4150 50  0001 C CNN
+F 0 "#PWR026" H 2350 4150 50  0001 C CNN
 F 1 "GND" H 2350 4250 50  0000 C CNN
 F 2 "" H 2350 4400 50  0000 C CNN

Commit message: исправление ошибок
Parts:
- removed C20: C, symbol C
- removed C3: 0.1U, symbol C
- added C? (x3): 0.1uF, symbol C
Connections:
- net labels added: +5V
- no-connect marks 11 -> 9

Commit message: Добавление WS2812, исправление всех замечаний
Parts:
- removed C13: C, symbol C
- removed C15: 0.1U, symbol C
- removed C16: 10U, symbol C
- removed FB1: L3, symbol INDUCTOR
- removed FB2: L4, symbol INDUCTOR
- removed FB3: L1, symbol INDUCTOR
- removed FB4: L2, symbol INDUCTOR
- added C?: 0.1uF, symbol C
- added R? (x2): 470, symbol R
- C18: value 10U -> 0.1uF
- C19, C4: value C -> 27pF
- U2, U3, U4: symbol PL2303 -> pl2303
- Y1: symbol CRYSTAL -> Crystal
- gave numbers to parts that had none: 3
Connections:
- net labels removed: GND_3V3, VCC, VDD, VDD_3V3, VDD_PLL
- wire segments 94 -> 84
Other:
- moved on the sheet: C17, C18, R3, R4, R5

Commit message: Изменения в CvPCB
Parts:
- removed P2: USB_A, symbol USB_A
- removed U3, U4: PL2303, symbol pl2303
- added P2: USB_OTG, Connect:USB_Micro-B, symbol USB_OTG
- C14, C17, C18, C3, C5, C6: footprint (none) -> Capacitors_SMD:C_0402
- C15: renamed from C?; footprint (none) -> Capacitors_SMD:C_0402
- C19, C4: footprint (none) -> Capacitors_SMD:C_0603_HandSoldering
- D1: footprint (none) -> LEDs:LED_0805
- D3: footprint (none) -> LEDs:LED-8MM
- R1, R2, R7, R8: footprint (none) -> Resistors_SMD:R_0805_HandSoldering
- R12, R13: renamed from R?; footprint (none) -> Resistors_SMD:R_0805_HandSoldering
- R3, R4, R5: footprint (none) -> Resistors_SMD:R_0402
- U2: footprint (none) -> Sockets:zip28
- Y1: footprint (none) -> Crystals:Crystal_FOX-FE_SMD
Connections:
- net +5V: now also P2.1 (VCC)
- net GND: now also P2.5 (GND)
- net at R3.2: now also P2.2 (D-)
- net at R4.2, R5.1: now also P2.3 (D+)
- no-connect marks 9 -> 10

Commit message: Небольшие изменения
Parts:
- U2: footprint Sockets:zip28 -> Housings_SSOP:SSOP-28_5.3x10.2mm_Pitch0.65mm
- Y1: footprint Crystals:Crystal_FOX-FE_SMD -> Crystals:Crystal_HC49-U_Vertical
Changed lines of the file:
@@
 F 0 "U2" H 3250 1550 60  0000 C CNN
 F 1 "PL2303" H 2950 3050 60  0000 C CNN
-F 2 "Sockets:zip28" H 2550 3300 60  0001 C CNN
+F 2 "Housings_SSOP:SSOP-28_5.3x10.2mm_Pitch0.65mm" H 2550 3300 60  0001 C CNN
 F 3 "" H 2550 3300 60  0000 C CNN
 	1    2550 3300
@@
 F 0 "Y1" H 950 3450 50  0000 C CNN
 F 1 "CRYSTAL" H 950 3150 50  0000 C CNN
-F 2 "Crystals:Crystal_FOX-FE_SMD" H 950 3300 50  0001 C CNN
+F 2 "Crystals:Crystal_HC49-U_Vertical" H 950 3300 50  0001 C CNN
 F 3 "" H 950 3300 50  0000 C CNN
 	1    950  3300
