File: pl2303.sch (KiCad schematic (older format))
At the start: 24 parts, among them P2 USB_OTG, U2 PL2303, Y1 CRYSTAL

Commit message: Последние изменения
Connections:
- net VCC is gone; now on net USB_IN: U2.20 (VDD), U2.24 (VDD_PLL), U2.8 (VDD)
Other:
- note added: "blah"
Changed lines of the file:
@@
 $EndComp
 $Comp
-L GND #PWR028
+L GND #PWR025
 U 1 1 5705278D
 P 9200 4000
-F 0 "#PWR028" H 9200 3750 50  0001 C CNN
+F 0 "#PWR025" H 9200 3750 50  0001 C CNN
 F 1 "GND" H 9200 3850 50  0000 C CNN
 F 2 "" H 9200 4000 50  0000 C CNN
@@
 $EndComp
 $Comp
-L GND #PWR029
+L GND #PWR026
 U 1 1 570529E3
 P 8500 5700
-F 0 "#PWR029" H 8500 5450 50  0001 C CNN
+F 0 "#PWR026" H 8500 5450 50  0001 C CNN
 F 1 "GND" H 8500 5550 50  0000 C CNN
 F 2 "" H 8500 5700 50  0000 C CNN
@@
 $EndComp
 $Comp
-L GND #PWR030
+L GND #PWR027
 U 1 1 570620C0
 P 2950 5500
-F 0 "#PWR030" H 2950 5250 50  0001 C CNN
+F 0 "#PWR027" H 2950 5250 50  0001 C CNN
 F 1 "GND" H 2950 5350 50  0000 C CNN
 F 2 "" H 2950 5500 50  0000 C CNN
@@
 $EndComp
 $Comp
-L GND #PWR031
+L GND #PWR028
 U 1 1 570D14D2
 P 950 3800
-F 0 "#PWR031" H 950 3550 50  0001 C CNN
+F 0 "#PWR028" H 950 3550 50  0001 C CNN
 F 1 "GND" H 950 3650 50  0000 C CNN
 F 2 "" H 950 3800 50  0000 C CNN
@@
 NoConn ~ 3550 3700
 $Comp
-L GND #PWR032
+L GND #PWR029
 U 1 1 570D2EBB
 P 2450 5100
-F 0 "#PWR032" H 2450 4850 50  0001 C CNN
+F 0 "#PWR029" H 2450 4850 50  0001 C CNN
 F 1 "GND" H 2450 4950 50  0000 C CNN
 F 2 "" H 2450 5100 50  0000 C CNN
@@
 $EndComp
 $Comp
-L GND #PWR033
+L GND #PWR030
 U 1 1 570D2F71
 P 4850 3050
-F 0 "#PWR033" H 4850 2800 50  0001 C CNN
+F 0 "#PWR030" H 4850 2800 50  0001 C CNN
 F 1 "GND" H 4850 2900 50  0000 C CNN
 F 2 "" H 4850 3050 50  0000 C CNN
@@
 $EndComp
 $Comp
-L +3.3V #PWR034
+L +3.3V #PWR031
 U 1 1 570D3933
 P 9200 2900
-F 0 "#PWR034" H 9200 2750 50  0001 C CNN
+F 0 "#PWR031" H 9200 2750 50  0001 C CNN
 F 1 "+3.3V" H 9200 3040 50  0000 C CNN
 F 2 "" H 9200 2900 50  0000 C CNN
@@
 $EndComp
 $Comp
-L +5V #PWR035
+L +5V #PWR032
 U 1 1 5717E4F4
 P 1195 890
-F 0 "#PWR035" H 1195 740 50  0001 C CNN
+F 0 "#PWR032" H 1195 740 50  0001 C CNN
 F 1 "+5V" H 1195 1030 50  0000 C CNN
 F 2 "" H 1195 890 50  0000 C CNN
@@
 $EndComp
 $Comp
-L GND #PWR036
+L GND #PWR033
 U 1 1 5717E503
 P 1195 1940
-F 0 "#PWR036" H 1195 1690 50  0001 C CNN
+F 0 "#PWR033" H 1195 1690 50  0001 C CNN
 F 1 "GND" H 1195 1790 50  0000 C CNN
 F 2 "" H 1195 1940 50  0000 C CNN
@@
 $EndComp
 $Comp
-L +5V #PWR037
+L +5V #PWR034
 U 1 1 5717F490
 P 2350 1650
-F 0 "#PWR037" H 2350 1500 50  0001 C CNN
+F 0 "#PWR034" H 2350 1500 50  0001 C CNN
 F 1 "+5V" H 2350 1790 50  0000 C CNN
 F 2 "" H 2350 1650 50  0000 C CNN
@@
 	8500 5000 8650 5000
 $Comp
-L +5V #PWR038
+L +5V #PWR035
 U 1 1 571E851C
 P 4600 1700
-F 0 "#PWR038" H 4600 1550 50  0001 C CNN
+F 0 "#PWR035" H 4600 1550 50  0001 C CNN
 F 1 "+5V" H 4600 1840 50  0000 C CNN
 F 2 "" H 4600 1700 50  0000 C CNN
@@
 	7700 5700 7700 5605
 $Comp
-L +3.3V #PWR039
+L +3.3V #PWR036
 U 1 1 574DBF4C
 P 7700 5605
-F 0 "#PWR039" H 7700 5455 50  0001 C CNN
+F 0 "#PWR036" H 7700 5455 50  0001 C CNN
 F 1 "+3.3V" H 7700 5745 50  0000 C CNN
 F 2 "" H 7700 5605 50  0000 C CNN
@@
 $EndComp
 $Comp
-L +3.3V #PWR040
+L +3.3V #PWR037
 U 1 1 574DC8B0
 P 2750 1460
-F 0 "#PWR040" H 2750 1310 50  0001 C CNN
+F 0 "#PWR037" H 2750 1310 50  0001 C CNN
 F 1 "+3.3V" H 2750 1600 50  0000 C CNN
 F 2 "" H 2750 1460 50  0000 C CNN
@@
 Wire Wire Line
 	7940 5100 7940 6050
-$Comp
-L VCC #PWR041
-U 1 1 578E507F
-P 2550 1535
-F 0 "#PWR041" H 2550 1385 50  0001 C CNN
-F 1 "VCC" H 2550 1685 50  0000 C CNN
-F 2 "" H 2550 1535 50  0000 C CNN
-F 3 "" H 2550 1535 50  0000 C CNN
-	1    2550 1535
-	1    0    0    -1
-$EndComp
 Wire Wire Line
 	8500 5000 8500 4465
 Wire Wire Line
 	2750 1460 2750 2300
+Text GLabel 2550 1535 1    60   Input ~ 0
+USB_IN
+Wire Notes Line
+	7870 1160 7870 2225
+Wire Notes Line
+	7870 2225 7855 2225
+Text Notes 7520 1295 0    60   ~ 0
+blah
 $EndSCHEMATC

Commit message: Точно последняя версия
Parts:
- P2: footprint Connect:USB_Micro-B -> open-project:MICRO-B_USB
Changed lines of the file:
@@
 LIBS:display
 LIBS:ws2812
+LIBS:open-project
 LIBS:cypress
 LIBS:siliconi
@@
 F 0 "P2" H 9275 5075 50  0000 C CNN
 F 1 "USB_OTG" H 8950 5400 50  0000 C CNN
-F 2 "Connect:USB_Micro-B" V 8900 5100 50  0001 C CNN
+F 2 "open-project:MICRO-B_USB" V 8900 5100 50  0001 C CNN
 F 3 "" V 8900 5100 50  0000 C CNN
 	1    8950 5200
