File: LM2596.sch (KiCad schematic (older format))
At the start: 8 parts

Commit message: Изменения футпринтов и расположения на плате
Parts:
- C2: footprint Capacitors_SMD:C_0402 -> Capacitors_SMD:C_0805
- L1: footprint Inductors:NR4018 -> INDUCTOR-12x12:INDUCTOR_12x12
- R14, R15: footprint Resistors_SMD:R_0402 -> Resistors_SMD:R_0805
Changed lines of the file:
@@
 $Descr A4 11693 8268
 encoding utf-8
-Sheet 2 4
+Sheet 4 4
 Title ""
 Date "20 apr 2016"
@@
 F 0 "C2" H 6350 3800 40  0000 L BNN
 F 1 "0.1uF" H 6356 3615 40  0000 L CNN
-F 2 "Capacitors_SMD:C_0402" V 6388 3550 30  0001 C CNN
+F 2 "Capacitors_SMD:C_0805" V 6388 3550 30  0001 C CNN
 F 3 "~" H 6350 3700 60  0000 C CNN
 	1    6350 3700
@@
 F 0 "L1" V 5350 3300 40  0000 C CNN
 F 1 "INDUCTOR" V 5500 3300 40  0000 C CNN
-F 2 "Inductors:NR4018" H 5400 3300 60  0001 C CNN
+F 2 "INDUCTOR-12x12:INDUCTOR_12x12" H 5400 3300 60  0001 C CNN
 F 3 "~" H 5400 3300 60  0000 C CNN
 	1    5400 3300
@@
 Vout
 $Comp
-L GND #PWR01
+L GND #PWR035
 U 1 1 56DED666
 P 6050 4200
-F 0 "#PWR01" H 6050 4200 30  0001 C CNN
+F 0 "#PWR035" H 6050 4200 30  0001 C CNN
 F 1 "GND" H 6050 4130 30  0001 C CNN
 F 2 "" H 6050 4200 60  0000 C CNN
@@
 $EndComp
 $Comp
-L GND #PWR02
+L GND #PWR036
 U 1 1 56DED66C
 P 8200 4300
-F 0 "#PWR02" H 8200 4300 30  0001 C CNN
+F 0 "#PWR036" H 8200 4300 30  0001 C CNN
 F 1 "GND" H 8200 4230 30  0001 C CNN
 F 2 "" H 8200 4300 60  0000 C CNN
@@
 F 0 "R14" V 8280 3450 50  0000 C CNN
 F 1 "1k" V 8200 3450 50  0000 C CNN
-F 2 "Resistors_SMD:R_0402" V 8130 3450 50  0001 C CNN
+F 2 "Resistors_SMD:R_0805" V 8130 3450 50  0001 C CNN
 F 3 "" H 8200 3450 50  0000 C CNN
 	1    8200 3450
@@
 F 0 "R15" V 8280 3950 50  0000 C CNN
 F 1 "1k" V 8200 3950 50  0000 C CNN
-F 2 "Resistors_SMD:R_0402" V 8130 3950 50  0001 C CNN
+F 2 "Resistors_SMD:R_0805" V 8130 3950 50  0001 C CNN
 F 3 "" H 8200 3950 50  0000 C CNN
 	1    8200 3950

Commit message: Питание и LM2596
Parts:
- added JP2: JUMPER, Connect:PINHEAD1-2, symbol JUMPER
- added R9: R, Resistors_SMD:R_0805, symbol R
- C1: footprint Capacitors_SMD:C_0805_HandSoldering -> Capacitors_ThroughHole:C_Radial_D7.5_L11.2_P2.5
- Cff1: footprint Capacitors_SMD:C_0603_HandSoldering -> Capacitors_ThroughHole:C_Radial_D6.3_L11.2_P2.5
Connections:
- net FB: now also JP2.1
- net GND: now also R9.2
- new net: JP2.2, R9.1
Changed lines of the file:
@@
 F 0 "Cff1" H 7750 3550 40  0000 L CNN
 F 1 "33nF" H 7756 3365 40  0000 L CNN
-F 2 "Capacitors_SMD:C_0603_HandSoldering" H 7788 3300 30  0001 C CNN
+F 2 "Capacitors_ThroughHole:C_Radial_D6.3_L11.2_P2.5" H 7788 3300 30  0001 C CNN
 F 3 "~" H 7750 3450 60  0000 C CNN
 	1    7750 3450
@@
 F 0 "C1" H 6050 3800 40  0000 L CNN
 F 1 "470uF" H 6056 3615 40  0000 L CNN
-F 2 "Capacitors_SMD:C_0805_HandSoldering" H 6088 3550 30  0000 C CNN
+F 2 "Capacitors_ThroughHole:C_Radial_D7.5_L11.2_P2.5" H 6088 3550 30  0000 C CNN
 F 3 "~" H 6050 3700 60  0000 C CNN
 	1    6050 3700
@@
 Connection ~ 7750 3150
 Wire Wire Line
-	7425 3700 8200 3700
+	7425 3700 8300 3700
 Wire Wire Line
 	7750 3600 7750 3700
@@
 L GND #PWR037
 U 1 1 56DED66C
-P 8200 4300
-F 0 "#PWR037" H 8200 4300 30  0001 C CNN
-F 1 "GND" H 8200 4230 30  0001 C CNN
-F 2 "" H 8200 4300 60  0000 C CNN
-F 3 "" H 8200 4300 60  0000 C CNN
-	1    8200 4300
+P 8650 4300
+F 0 "#PWR037" H 8650 4300 30  0001 C CNN
+F 1 "GND" H 8650 4230 30  0001 C CNN
+F 2 "" H 8650 4300 60  0000 C CNN
+F 3 "" H 8650 4300 60  0000 C CNN
+	1    8650 4300
 	1    0    0    -1
 $EndComp
-Wire Wire Line
-	8200 4100 8200 4300
 Text HLabel 4500 3600 2    60   Input ~ 0
 CS
@@
 	8200 3600 8200 3800
 Connection ~ 8200 3700
+$Comp
+L JUMPER JP2
+U 1 1 57404772
+P 8600 3700
+F 0 "JP2" H 8600 3850 50  0000 C CNN
+F 1 "JUMPER" H 8600 3620 50  0000 C CNN
+F 2 "Connect:PINHEAD1-2" H 8600 3700 50  0001 C CNN
+F 3 "" H 8600 3700 50  0000 C CNN
+	1    8600 3700
+	1    0    0    -1
+$EndComp
+$Comp
+L R R9
+U 1 1 5740479F
+P 9000 3950
+F 0 "R9" V 9080 3950 50  0000 C CNN
+F 1 "R" V 9000 3950 50  0000 C CNN
+F 2 "Resistors_SMD:R_0805" V 8930 3950 50  0001 C CNN
+F 3 "" H 9000 3950 50  0000 C CNN
+	1    9000 3950
+	1    0    0    -1
+$EndComp
+Wire Wire Line
+	8900 3700 9000 3700
+Wire Wire Line
+	9000 3700 9000 3800
+Wire Wire Line
+	9000 4200 9000 4100
+Wire Wire Line
+	8200 4200 9000 4200
+Wire Wire Line
+	8650 4200 8650 4300
+Wire Wire Line
+	8200 4100 8200 4200
+Connection ~ 8650 4200
 $EndSCHEMATC

Commit message: исправления
Parts:
- Cff1: footprint Capacitors_ThroughHole:C_Radial_D6.3_L11.2_P2.5 -> Capacitors_SMD:C_0805
Changed lines of the file:
@@
 F 0 "Cff1" H 7750 3550 40  0000 L CNN
 F 1 "33nF" H 7756 3365 40  0000 L CNN
-F 2 "Capacitors_ThroughHole:C_Radial_D6.3_L11.2_P2.5" H 7788 3300 30  0001 C CNN
+F 2 "Capacitors_SMD:C_0805" H 7788 3300 30  0001 C CNN
 F 3 "~" H 7750 3450 60  0000 C CNN
 	1    7750 3450

Commit message: LM2596
Parts:
- removed JP2: JUMPER, Connect:PINHEAD1-2, symbol JUMPER
- added JP?: JUMPER3, symbol JUMPER3
Connections:
- net FB: no longer R14.2, R15.1
- new net: JP?.1, R14.2
Other:
- moved on the sheet: R15, R9
Changed lines of the file:
@@
 	1    0    0    -1
 $EndComp
-Wire Wire Line
-	4500 3300 5100 3300
-Wire Wire Line
-	5700 3300 6650 3300
-Wire Wire Line
-	6050 3300 6050 3550
-Wire Wire Line
-	6350 3150 6350 3550
-Connection ~ 6050 3300
-Wire Wire Line
-	7750 3150 7750 3300
-Wire Wire Line
-	6350 3150 8200 3150
-Connection ~ 6350 3300
-Connection ~ 7750 3150
-Wire Wire Line
-	7425 3700 8300 3700
-Wire Wire Line
-	7750 3600 7750 3700
-Connection ~ 7750 3700
-Wire Wire Line
-	4900 4100 4900 3900
-Connection ~ 3900 4100
-Wire Wire Line
-	4900 3500 4900 3300
-Connection ~ 4900 3300
-Wire Wire Line
-	6050 3850 6050 4200
-Connection ~ 4900 4100
-Wire Wire Line
-	6350 4100 6350 3850
-Connection ~ 6050 4100
-Wire Wire Line
-	2800 3450 3100 3450
 Text HLabel 2800 3450 0    60   Input ~ 0
 Vin
@@
 L GND #PWR037
 U 1 1 56DED66C
-P 8650 4300
-F 0 "#PWR037" H 8650 4300 30  0001 C CNN
-F 1 "GND" H 8650 4230 30  0001 C CNN
-F 2 "" H 8650 4300 60  0000 C CNN
-F 3 "" H 8650 4300 60  0000 C CNN
-	1    8650 4300
+P 8655 4810
+F 0 "#PWR037" H 8655 4810 30  0001 C CNN
+F 1 "GND" H 8655 4740 30  0001 C CNN
+F 2 "" H 8655 4810 60  0000 C CNN
+F 3 "" H 8655 4810 60  0000 C CNN
+	1    8655 4810
 	1    0    0    -1
 $EndComp
@@
 	1    0    0    -1
 $EndComp
-Wire Wire Line
-	3900 4100 6350 4100
 $Comp
 L R R14
@@
 L R R15
 U 1 1 572B2E55
-P 8200 3950
-F 0 "R15" V 8280 3950 50  0000 C CNN
-F 1 "1k" V 8200 3950 50  0000 C CNN
-F 2 "Resistors_SMD:R_0805" V 8130 3950 50  0001 C CNN
-F 3 "" H 8200 3950 50  0000 C CNN
-	1    8200 3950
-	1    0    0    -1
-$EndComp
-Wire Wire Line
-	8200 3150 8200 3300
-Wire Wire Line
-	8200 3600 8200 3800
-Connection ~ 8200 3700
-$Comp
-L JUMPER JP2
-U 1 1 57404772
-P 8600 3700
-F 0 "JP2" H 8600 3850 50  0000 C CNN
-F 1 "JUMPER" H 8600 3620 50  0000 C CNN
-F 2 "Connect:PINHEAD1-2" H 8600 3700 50  0001 C CNN
-F 3 "" H 8600 3700 50  0000 C CNN
-	1    8600 3700
+P 8205 4460
+F 0 "R15" V 8285 4460 50  0000 C CNN
+F 1 "1k" V 8205 4460 50  0000 C CNN
+F 2 "Resistors_SMD:R_0805" V 8135 4460 50  0001 C CNN
+F 3 "" H 8205 4460 50  0000 C CNN
+	1    8205 4460
 	1    0    0    -1
 $EndComp
@@
 L R R9
 U 1 1 5740479F
-P 9000 3950
-F 0 "R9" V 9080 3950 50  0000 C CNN
-F 1 "R" V 9000 3950 50  0000 C CNN
-F 2 "Resistors_SMD:R_0805" V 8930 3950 50  0001 C CNN
-F 3 "" H 9000 3950 50  0000 C CNN
-	1    9000 3950
+P 9005 4460
+F 0 "R9" V 9085 4460 50  0000 C CNN
+F 1 "R" V 9005 4460 50  0000 C CNN
+F 2 "Resistors_SMD:R_0805" V 8935 4460 50  0001 C CNN
+F 3 "" H 9005 4460 50  0000 C CNN
+	1    9005 4460
 	1    0    0    -1
 $EndComp
+$Comp
+L JUMPER3 JP?
+U 1 1 5740CAA4
+P 8205 3995
+F 0 "JP?" H 8255 3895 50  0000 L CNN
+F 1 "JUMPER3" H 8205 4095 50  0000 C BNN
+F 2 "" H 8205 3995 50  0000 C CNN
+F 3 "" H 8205 3995 50  0000 C CNN
+	1    8205 3995
+	0    1    1    0
+$EndComp
 Wire Wire Line
-	8900 3700 9000 3700
+	4500 3300 4900 3300
 Wire Wire Line
-	9000 3700 9000 3800
+	4900 3300 5100 3300
 Wire Wire Line
-	9000 4200 9000 4100
+	5700 3300 6050 3300
 Wire Wire Line
-	8200 4200 9000 4200
+	6050 3300 6350 3300
 Wire Wire Line
-	8650 4200 8650 4300
+	6350 3300 6650 3300
 Wire Wire Line
-	8200 4100 8200 4200
-Connection ~ 8650 4200
+	6050 3300 6050 3550
+Wire Wire Line
+	6350 3150 6350 3300
+Wire Wire Line
+	6350 3300 6350 3550
+Connection ~ 6050 3300
+Wire Wire Line
+	7750 3150 7750 3300
+Wire Wire Line
+	6350 3150 7750 3150
+Wire Wire Line
+	7750 3150 8200 3150
+Connection ~ 6350 3300
+Connection ~ 7750 3150
+Wire Wire Line
+	7425 3700 7750 3700
+Wire Wire Line
+	7750 3700 7750 3600
+Connection ~ 7750 3700
+Wire Wire Line
+	4900 4100 4900 3900
+Connection ~ 3900 4100
+Wire Wire Line
+	4900 3500 4900 3300
+Connection ~ 4900 3300
+Wire Wire Line
+	6050 3850 6050 4100
+Wire Wire Line
+	6050 4100 6050 4200
+Connection ~ 4900 4100
+Wire Wire Line
+	6350 4100 6350 3850
+Connection ~ 6050 4100
+Wire Wire Line
+	2800 3450 3100 3450
+Wire Wire Line
+	3900 4100 4900 4100
+Wire Wire Line
+	4900 4100 6050 4100
+Wire Wire Line
+	6050 4100 6350 4100
+Wire Wire Line
+	8200 3150 8200 3300
+Wire Wire Line
+	9005 4710 9005 4610
+Wire Wire Line
+	8205 4710 8655 4710
+Wire Wire Line
+	8655 4710 9005 4710
+Wire Wire Line
+	8655 4710 8655 4810
+Wire Wire Line
+	8205 4610 8205 4710
+Connection ~ 8655 4710
+Wire Wire Line
+	8200 3600 8200 3745
+Wire Wire Line
+	8200 3745 8205 3745
 $EndSCHEMATC

Commit message: исправлена LM2596
Parts:
- JP2: renamed from JP?; footprint (none) -> Connect:PINHEAD1-3
Connections:
- wire segments 30 -> 23
Other:
- moved on the sheet: JP2
Changed lines of the file:
@@
-	1    0    0    -1
-$EndComp
-$Comp
-L GND #PWR037
-U 1 1 56DED66C
-P 8655 4810
-F 0 "#PWR037" H 8655 4810 30  0001 C CNN
-F 1 "GND" H 8655 4740 30  0001 C CNN
-F 2 "" H 8655 4810 60  0000 C CNN
-F 3 "" H 8655 4810 60  0000 C CNN
-	1    8655 4810
 	1    0    0    -1
 $EndComp
@@
 L R R15
 U 1 1 572B2E55
-P 8205 4460
-F 0 "R15" V 8285 4460 50  0000 C CNN
-F 1 "1k" V 8205 4460 50  0000 C CNN
-F 2 "Resistors_SMD:R_0805" V 8135 4460 50  0001 C CNN
-F 3 "" H 8205 4460 50  0000 C CNN
-	1    8205 4460
+P 8200 4460
+F 0 "R15" V 8280 4460 50  0000 C CNN
+F 1 "1k" V 8200 4460 50  0000 C CNN
+F 2 "Resistors_SMD:R_0805" V 8130 4460 50  0001 C CNN
+F 3 "" H 8200 4460 50  0000 C CNN
+	1    8200 4460
 	1    0    0    -1
 $EndComp
@@
 L R R9
 U 1 1 5740479F
-P 9005 4460
-F 0 "R9" V 9085 4460 50  0000 C CNN
-F 1 "R" V 9005 4460 50  0000 C CNN
-F 2 "Resistors_SMD:R_0805" V 8935 4460 50  0001 C CNN
-F 3 "" H 9005 4460 50  0000 C CNN
-	1    9005 4460
+P 9000 4460
+F 0 "R9" V 9080 4460 50  0000 C CNN
+F 1 "R" V 9000 4460 50  0000 C CNN
+F 2 "Resistors_SMD:R_0805" V 8930 4460 50  0001 C CNN
+F 3 "" H 9000 4460 50  0000 C CNN
+	1    9000 4460
 	1    0    0    -1
 $EndComp
 $Comp
-L JUMPER3 JP?
+L JUMPER3 JP2
 U 1 1 5740CAA4
-P 8205 3995
-F 0 "JP?" H 8255 3895 50  0000 L CNN
-F 1 "JUMPER3" H 8205 4095 50  0000 C BNN
-F 2 "" H 8205 3995 50  0000 C CNN
-F 3 "" H 8205 3995 50  0000 C CNN
-	1    8205 3995
-	0    1    1    0
+P 8200 4000
+F 0 "JP2" H 8250 3900 50  0000 L CNN
+F 1 "JUMPER3" H 8200 4100 50  0000 C BNN
+F 2 "Connect:PINHEAD1-3" H 8200 4000 50  0001 C CNN
+F 3 "" H 8200 4000 50  0000 C CNN
+	1    8200 4000
+	0    -1   -1   0
 $EndComp
 Wire Wire Line
-	4500 3300 4900 3300
+	4500 3300 5100 3300
 Wire Wire Line
-	4900 3300 5100 3300
-Wire Wire Line
-	5700 3300 6050 3300
-Wire Wire Line
-	6050 3300 6350 3300
-Wire Wire Line
-	6350 3300 6650 3300
+	5700 3300 6650 3300
 Wire Wire Line
 	6050 3300 6050 3550
 Wire Wire Line
-	6350 3150 6350 3300
-Wire Wire Line
-	6350 3300 6350 3550
+	6350 3150 6350 3550
 Connection ~ 6050 3300
 Wire Wire Line
 	7750 3150 7750 3300
 Wire Wire Line
-	6350 3150 7750 3150
-Wire Wire Line
-	7750 3150 8200 3150
+	6350 3150 8200 3150
 Connection ~ 6350 3300
 Connection ~ 7750 3150
 Wire Wire Line
-	7425 3700 7750 3700
+	7425 3700 8200 3700
 Wire Wire Line
 	7750 3700 7750 3600
@@
 Connection ~ 4900 3300
 Wire Wire Line
-	6050 3850 6050 4100
-Wire Wire Line
-	6050 4100 6050 4200
+	6050 3850 6050 4200
 Connection ~ 4900 4100
 Wire Wire Line
@@
 	2800 3450 3100 3450
 Wire Wire Line
-	3900 4100 4900 4100
-Wire Wire Line
-	4900 4100 6050 4100
-Wire Wire Line
-	6050 4100 6350 4100
+	3900 4100 6350 4100
 Wire Wire Line
 	8200 3150 8200 3300
 Wire Wire Line
-	9005 4710 9005 4610
+	8200 3600 8200 3755
+Connection ~ 8200 3700
 Wire Wire Line
-	8205 4710 8655 4710
+	8200 4250 8200 4310
 Wire Wire Line
-	8655 4710 9005 4710
+	8200 4610 8200 4680
 Wire Wire Line
-	8655 4710 8655 4810
+	8200 4680 9000 4680
 Wire Wire Line
-	8205 4610 8205 4710
-Connection ~ 8655 4710
+	9000 4680 9000 4610
 Wire Wire Line
-	8200 3600 8200 3745
+	9000 4310 9000 4000
 Wire Wire Line
-	8200 3745 8205 3745
+	9000 4000 8300 4000
+Wire Wire Line
+	8625 4680 8625 4755
+Connection ~ 8625 4680
+$Comp
+L GND #PWR037
+U 1 1 57477506
+P 8625 4755
+F 0 "#PWR037" H 8625 4505 50  0001 C CNN
+F 1 "GND" H 8625 4605 50  0000 C CNN
+F 2 "" H 8625 4755 50  0000 C CNN
+F 3 "" H 8625 4755 50  0000 C CNN
+	1    8625 4755
+	1    0    0    -1
+$EndComp
 $EndSCHEMATC

Commit message: Небольшие изменения
Changed lines of the file:
@@
 L JUMPER3 JP2
 U 1 1 5740CAA4
-P 8200 4000
-F 0 "JP2" H 8250 3900 50  0000 L CNN
-F 1 "JUMPER3" H 8200 4100 50  0000 C BNN
-F 2 "Connect:PINHEAD1-3" H 8200 4000 50  0001 C CNN
-F 3 "" H 8200 4000 50  0000 C CNN
-	1    8200 4000
+P 8200 4005
+F 0 "JP2" H 8250 3905 50  0000 L CNN
+F 1 "JUMPER3" H 8200 4105 50  0000 C BNN
+F 2 "Connect:PINHEAD1-3" H 8200 4005 50  0001 C CNN
+F 3 "" H 8200 4005 50  0000 C CNN
+	1    8200 4005
 	0    -1   -1   0
 $EndComp
@@
 Connection ~ 8200 3700
 Wire Wire Line
-	8200 4250 8200 4310
+	8200 4255 8200 4310
 Wire Wire Line
 	8200 4610 8200 4680
@@
 	9000 4310 9000 4000
 Wire Wire Line
-	9000 4000 8300 4000
+	9000 4000 8300 4005
 Wire Wire Line
 	8625 4680 8625 4755

Commit message: Готовая плата версия_1
Connections:
- net FB: now also JP2.2; no longer JP2.3
- net at R15.1: now also JP2.3; no longer JP2.1
- net at R9.1: now also JP2.1; no longer JP2.2
Other:
- moved on the sheet: JP2, R14
Changed lines of the file:
@@
 LIBS:Pulse_Module-rescue
 LIBS:conn3
-LIBS:pl2303
 LIBS:power
 LIBS:device
@@
 L R R14
 U 1 1 572B2DAD
-P 8200 3450
-F 0 "R14" V 8280 3450 50  0000 C CNN
-F 1 "1k" V 8200 3450 50  0000 C CNN
-F 2 "Resistors_SMD:R_0805" V 8130 3450 50  0001 C CNN
-F 3 "" H 8200 3450 50  0000 C CNN
-	1    8200 3450
+P 8040 3460
+F 0 "R14" V 8120 3460 50  0000 C CNN
+F 1 "1k" V 8040 3460 50  0000 C CNN
+F 2 "Resistors_SMD:R_0805" V 7970 3460 50  0001 C CNN
+F 3 "" H 8040 3460 50  0000 C CNN
+	1    8040 3460
 	1    0    0    -1
 $EndComp
@@
 F 3 "" H 8200 4005 50  0000 C CNN
 	1    8200 4005
-	0    -1   -1   0
-$EndComp
-Wire Wire Line
-	4500 3300 5100 3300
-Wire Wire Line
-	5700 3300 6650 3300
-Wire Wire Line
-	6050 3300 6050 3550
-Wire Wire Line
-	6350 3150 6350 3550
-Connection ~ 6050 3300
-Wire Wire Line
-	7750 3150 7750 3300
-Wire Wire Line
-	6350 3150 8200 3150
-Connection ~ 6350 3300
-Connection ~ 7750 3150
-Wire Wire Line
-	7425 3700 8200 3700
-Wire Wire Line
-	7750 3700 7750 3600
-Connection ~ 7750 3700
-Wire Wire Line
-	4900 4100 4900 3900
-Connection ~ 3900 4100
-Wire Wire Line
-	4900 3500 4900 3300
-Connection ~ 4900 3300
-Wire Wire Line
-	6050 3850 6050 4200
-Connection ~ 4900 4100
-Wire Wire Line
-	6350 4100 6350 3850
-Connection ~ 6050 4100
-Wire Wire Line
-	2800 3450 3100 3450
-Wire Wire Line
-	3900 4100 6350 4100
-Wire Wire Line
-	8200 3150 8200 3300
-Wire Wire Line
-	8200 3600 8200 3755
-Connection ~ 8200 3700
-Wire Wire Line
-	8200 4255 8200 4310
-Wire Wire Line
-	8200 4610 8200 4680
-Wire Wire Line
-	8200 4680 9000 4680
-Wire Wire Line
-	9000 4680 9000 4610
-Wire Wire Line
-	9000 4310 9000 4000
-Wire Wire Line
-	9000 4000 8300 4005
-Wire Wire Line
-	8625 4680 8625 4755
-Connection ~ 8625 4680
+	0    1    1    0
+$EndComp
 $Comp
 L GND #PWR037
@@
 	1    0    0    -1
 $EndComp
+Wire Wire Line
+	4500 3300 5100 3300
+Wire Wire Line
+	5700 3300 6650 3300
+Wire Wire Line
+	6050 3300 6050 3550
+Wire Wire Line
+	6350 3150 6350 3550
+Connection ~ 6050 3300
+Wire Wire Line
+	7750 3150 7750 3300
+Wire Wire Line
+	6350 3150 8040 3150
+Connection ~ 6350 3300
+Connection ~ 7750 3150
+Wire Wire Line
+	4900 4100 4900 3900
+Connection ~ 3900 4100
+Wire Wire Line
+	4900 3500 4900 3300
+Connection ~ 4900 3300
+Wire Wire Line
+	6050 3850 6050 4200
+Connection ~ 4900 4100
+Wire Wire Line
+	6350 4100 6350 3850
+Connection ~ 6050 4100
+Wire Wire Line
+	2800 3450 3100 3450
+Wire Wire Line
+	3900 4100 6350 4100
+Wire Wire Line
+	8200 4255 8200 4310
+Wire Wire Line
+	8200 4610 8200 4680
+Wire Wire Line
+	8200 4680 9000 4680
+Wire Wire Line
+	9000 4680 9000 4610
+Wire Wire Line
+	9000 3755 9000 4310
+Wire Wire Line
+	8625 4680 8625 4755
+Connection ~ 8625 4680
+Wire Wire Line
+	8040 3150 8040 3310
+Wire Wire Line
+	8040 3610 8040 4005
+Wire Wire Line
+	8040 4005 8100 4005
+Wire Wire Line
+	7425 3700 8040 3700
+Connection ~ 8040 3700
+Wire Wire Line
+	7750 3600 7750 3700
+Connection ~ 7750 3700
+Wire Wire Line
+	8200 3755 9000 3755
 $EndSCHEMATC
